Commit message: start base of scte2.0 bot urdf and getting it to show up in rviz

File: sctebot2_description/urdf/standard/sctebot2.urdf.xacro (robot description, xacro)
@@ -2,10 +2,27 @@
 <robot name="sctebot2" xmlns:xacro="http://ros.org/wiki/xacro">
     <!-- URDF Tutorial https://docs.ros.org/en/rolling/Tutorials/Intermediate/URDF/Building-a-Visual-Robot-Model-with-URDF-from-Scratch.html -->
+    <!-- Robot base dimensions -->
+    <xacro:property name="base_length" value="0.442" /> <!-- wheel base derived from this -->
+    <xacro:property name="base_width" value="0.157" /> <!-- wheel track derived from this -->
+    <xacro:property name="base_height" value="0.01" />
     <link name="base_link">
         <visual>
+            <origin xyz="0 0 0" rpy="0 0 0"/>
             <geometry>
-                <cylinder length="0.6" radius="0.2"/>
+                <box size="${base_length} ${base_width} ${base_height}"/>
             </geometry>
         </visual>
+        <collision>
+            <origin xyz="0 0 0" rpy="0 0 0"/>
+            <geometry>
+                <box size="${base_length} ${base_width} ${base_height}"/>
+            </geometry>
+        </collision>
     </link>
+    <link name="base_footprint"/>
+    <joint name="base_footprint_joint" type="fixed">
+        <origin xyz="0 0 0" rpy="0 0 0"/>
+        <parent link="base_link"/>
+        <child link="base_footprint"/>
+    </joint>
 </robot>

Commit message: add color to help distinguish the body from everything else

File: sctebot2_description/urdf/standard/sctebot2.urdf.xacro (robot description, xacro)
@@ -6,4 +6,7 @@
     <xacro:property name="base_width" value="0.157" /> <!-- wheel track derived from this -->
     <xacro:property name="base_height" value="0.01" />
+    <material name="blue">
+        <color rgba="0 0 0.8 1"/>
+    </material>
     <link name="base_link">
         <visual>
@@ -12,4 +15,5 @@
                 <box size="${base_length} ${base_width} ${base_height}"/>
             </geometry>
+            <material name="blue"/>
         </visual>
         <collision>

Commit message: add wheels and bumpers to model

File: sctebot2_description/urdf/standard/sctebot2.urdf.xacro (robot description, xacro)
@@ -1,12 +1,50 @@
 <?xml version="1.0" ?>
 <robot name="sctebot2" xmlns:xacro="http://ros.org/wiki/xacro">
-    <!-- URDF Tutorial https://docs.ros.org/en/rolling/Tutorials/Intermediate/URDF/Building-a-Visual-Robot-Model-with-URDF-from-Scratch.html -->
+    <!--
+    URDF Tutorial https://docs.ros.org/en/humble/Tutorials/Intermediate/URDF/Building-a-Visual-Robot-Model-with-URDF-from-Scratch.html
+    ROS2 Control https://control.ros.org/humble/index.html
+     -->
+    <!-- Math constants -->
+    <xacro:property name="deg_to_rad" value="0.01745329251994329577"/>
+    <!-- materials -->
+    <material name="black_front">
+        <color rgba="0.1 0.1 0.1 1"/>
+    </material>
+    <material name="black_rear">
+        <color rgba="0.3 0.3 0.3 1"/>
+    </material>
+    <material name="red">
+        <color rgba="0.8 0 0.0 1"/>
+    </material>
+    <material name="blue">
+        <color rgba="0 0 0.8 1"/>
+    </material>
+    <material name="green">
+        <color rgba="0 0.8 0 1"/>
+    </material>
     <!-- Robot base dimensions -->
     <xacro:property name="base_length" value="0.442" /> <!-- wheel base derived from this -->
     <xacro:property name="base_width" value="0.157" /> <!-- wheel track derived from this -->
     <xacro:property name="base_height" value="0.01" />
-    <material name="blue">
-        <color rgba="0 0 0.8 1"/>
-    </material>
+    <xacro:property name="wheel_track" value="0.25"/>
+    <xacro:property name="wheel_base" value="0.33"/>
+    <xacro:property name="wheel_axis_height" value="0.05" />
+    <xacro:property name="wheel_radius" value="0.0525"/>
+    <xacro:property name="wheel_height" value="0.045"/>
+    <!-- base links -->
+    <link name="base_footprint">
+        <visual>
+            <origin xyz="0 0 0" rpy="0 0 0"/>
+            <geometry>
+                <box size="${base_length} ${base_width} ${base_height}"/>
+            </geometry>
+            <material name="green"/>
+        </visual>
+    </link>
+    <joint name="base_footprint_joint" type="fixed">
+        <origin xyz="0 0 -${wheel_axis_height}" rpy="0 0 0"/>
+        <parent link="base_link"/>
+        <child link="base_footprint"/>
+    </joint>
     <link name="base_link">
         <visual>
@@ -24,9 +62,131 @@
         </collision>
     </link>
-    <link name="base_footprint"/>
-    <joint name="base_footprint_joint" type="fixed">
-        <origin xyz="0 0 0" rpy="0 0 0"/>
+    <!-- bumpers -->
+    <xacro:property name="front_bumper_offset" value="0.075"/>
+    <xacro:property name="front_bumper_width" value="0.18"/>
+    <xacro:property name="front_bumper_height" value="0.07"/>
+    <link name="front_bumper">
+        <visual>
+            <origin xyz="0 0 0" rpy="0 0 0"/>
+            <geometry>
+                <box size="0.01 ${front_bumper_width} ${front_bumper_height}"/>
+            </geometry>
+            <material name="green"/>
+        </visual>
+        <collision>
+            <origin xyz="0 0 0" rpy="0 0 0"/>
+            <geometry>
+                <box size="0.01 ${front_bumper_width} ${front_bumper_height}"/>
+            </geometry>
+        </collision>
+    </link>
+    <joint name="front_bumper_joint" type="fixed">
+        <origin xyz="${front_bumper_offset + base_length / 2.0} 0 ${front_bumper_height / 2.0}" rpy="0 0 0"/>
         <parent link="base_link"/>
-        <child link="base_footprint"/>
+        <child link="front_bumper"/>
+    </joint>
+    <xacro:property name="rear_bumper_offset" value="0.065"/>
+    <xacro:property name="rear_bumper_width" value="0.255"/>
+    <xacro:property name="rear_bumper_height" value="0.07"/>
+    <link name="rear_bumper">
+        <visual>
+            <origin xyz="0 0 0" rpy="0 0 0"/>
+            <geometry>
+                <box size="0.01 ${rear_bumper_width} ${rear_bumper_height}"/>
+            </geometry>
+            <material name="red"/>
+        </visual>
+        <collision>
+            <origin xyz="0 0 0" rpy="0 0 0"/>
+            <geometry>
+                <box size="0.01 ${rear_bumper_width} ${rear_bumper_height}"/>
+            </geometry>
+        </collision>
+    </link>
+    <joint name="rear_bumper_joint" type="fixed">
+        <origin xyz="-${rear_bumper_offset + base_length / 2.0} 0 ${rear_bumper_height / 2.0}" rpy="0 0 0"/>
+        <parent link="base_link"/>
+        <child link="rear_bumper"/>
+    </joint>
+    <!-- wheels -->
+    <link name="left_front_wheel">
+        <visual>
+            <origin xyz="0 0 0" rpy="0 0 0"/>
+            <geometry>
+                <cylinder length="${wheel_height}" radius="${wheel_radius}"/>
+            </geometry>
+            <material name="black_front"/>
+        <collision>
+            <origin xyz="0 0 0" rpy="0 0 0"/>
+            <geometry>
+                <cylinder length="${wheel_height}" radius="${wheel_radius}"/>
+            </geometry>
+        </collision>
+        </visual>
+    </link>
+    <joint name="left_front_wheel_joint" type="fixed">
+        <origin xyz="${wheel_base / 2.0} ${wheel_track / 2.0} 0" rpy="${90 * deg_to_rad} 0 0" />
+        <parent link="base_link"/>
+        <child link="left_front_wheel"/>
+    </joint>
+    <link name="right_front_wheel">
+        <visual>
+            <origin xyz="0 0 0" rpy="0 0 0"/>
+            <geometry>
+                <cylinder length="${wheel_height}" radius="${wheel_radius}"/>
+            </geometry>
+            <material name="black_front"/>
+        <collision>
+            <origin xyz="0 0 0" rpy="0 0 0"/>
+            <geometry>
+                <cylinder length="${wheel_height}" radius="${wheel_radius}"/>
+            </geometry>
+        </collision>
+        </visual>
+    </link>
+    <joint name="right_front_wheel_joint" type="fixed">
+        <origin xyz="${wheel_base / 2.0} -${wheel_track / 2.0} 0" rpy="${90 * deg_to_rad} 0 0" />
+        <parent link="base_link"/>
+        <child link="right_front_wheel"/>
+    </joint>
+    <link name="left_rear_wheel">
+        <visual>
+            <origin xyz="0 0 0" rpy="0 0 0"/>
+            <geometry>
+                <cylinder length="${wheel_height}" radius="${wheel_radius}"/>
+            </geometry>
+            <material name="black_rear"/>
+        <collision>
+            <origin xyz="0 0 0" rpy="0 0 0"/>
+            <geometry>
+                <cylinder length="${wheel_height}" radius="${wheel_radius}"/>
+            </geometry>
+        </collision>
+        </visual>
+    </link>
+    <joint name="left_rear_wheel_joint" type="fixed">
+        <origin xyz="-${wheel_base / 2.0} ${wheel_track / 2.0} 0" rpy="${90 * deg_to_rad} 0 0" />
+        <parent link="base_link"/>
+        <child link="left_rear_wheel"/>
+    </joint>
+    <link name="right_rear_wheel">
+        <visual>
+            <origin xyz="0 0 0" rpy="0 0 0"/>
+            <geometry>
+                <cylinder length="${wheel_height}" radius="${wheel_radius}"/>
+            </geometry>
+            <material name="black_rear"/>
+        <collision>
+            <origin xyz="0 0 0" rpy="0 0 0"/>
+            <geometry>
+                <cylinder length="${wheel_height}" radius="${wheel_radius}"/>
+            </geometry>
+        </collision>
+        </visual>
+    </link>
+    <joint name="right_rear_wheel_joint" type="fixed">
+        <origin xyz="-${wheel_base / 2.0} -${wheel_track / 2.0} 0" rpy="${90 * deg_to_rad} 0 0" />
+        <parent link="base_link"/>
+        <child link="right_rear_wheel"/>
     </joint>
 </robot>

Commit message: add urdf models for lidar and realsense camera. Change wheel joints to be continous. Added joint_state_publisher_gui to launch although sometimes does not attach to wheels

File: sctebot2_description/urdf/standard/sctebot2.urdf.xacro (robot description, xacro)
@@ -4,4 +4,5 @@
     URDF Tutorial https://docs.ros.org/en/humble/Tutorials/Intermediate/URDF/Building-a-Visual-Robot-Model-with-URDF-from-Scratch.html
     ROS2 Control https://control.ros.org/humble/index.html
+    R2D2 https://github.com/ros/urdf_tutorial/tree/ros2
      -->
     <!-- Math constants -->
@@ -109,4 +110,5 @@
         <child link="rear_bumper"/>
     </joint>
+    <!-- end bumpbers -->
     <!-- wheels -->
     <link name="left_front_wheel">
@@ -125,5 +127,6 @@
         </visual>
     </link>
-    <joint name="left_front_wheel_joint" type="fixed">
+    <joint name="left_front_wheel_joint" type="continuous">
+        <axis xyz="0 0 1"/>
         <origin xyz="${wheel_base / 2.0} ${wheel_track / 2.0} 0" rpy="${90 * deg_to_rad} 0 0" />
         <parent link="base_link"/>
@@ -145,5 +148,6 @@
         </visual>
     </link>
-    <joint name="right_front_wheel_joint" type="fixed">
+    <joint name="right_front_wheel_joint" type="continuous">
+        <axis xyz="0 0 1"/>
         <origin xyz="${wheel_base / 2.0} -${wheel_track / 2.0} 0" rpy="${90 * deg_to_rad} 0 0" />
         <parent link="base_link"/>
@@ -165,5 +169,6 @@
         </visual>
     </link>
-    <joint name="left_rear_wheel_joint" type="fixed">
+    <joint name="left_rear_wheel_joint" type="continuous">
+        <axis xyz="0 0 1"/>
         <origin xyz="-${wheel_base / 2.0} ${wheel_track / 2.0} 0" rpy="${90 * deg_to_rad} 0 0" />
         <parent link="base_link"/>
@@ -185,8 +190,32 @@
         </visual>
     </link>
-    <joint name="right_rear_wheel_joint" type="fixed">
+    <joint name="right_rear_wheel_joint" type="continuous">
+        <axis xyz="0 0 1"/>
         <origin xyz="-${wheel_base / 2.0} -${wheel_track / 2.0} 0" rpy="${90 * deg_to_rad} 0 0" />
         <parent link="base_link"/>
         <child link="right_rear_wheel"/>
     </joint>
+    <!-- end wheels -->
+    <!-- sensors -->
+    <!-- x 0.323m span, 0.162m center from axis z -->
+    <link name="ydlidar_sensor">
+        <visual>
+            <origin xyz="0 0 0.3" rpy="0 0 0"/>
+            <geometry>
+                <!--cylinder length="0.041" radius="0.035"/-->
+                <mesh filename="package://ydlidar_description/meshes/ydlidar.dae"/>
+            </geometry>
+        </visual>
+    </link>
+    <joint name="ydlidar_sensor_joint" type="fixed">
+        <origin xyz="0 0 0" rpy="0 0 0"/>
+        <parent link="base_link"/>
+        <child link="ydlidar_sensor"/>
+    </joint>
+    <xacro:include filename="$(find realsense2_description)/urdf/_d455.urdf.xacro"/>
+    <xacro:arg name="use_nominal_extrinsics" default="false"/>
+    <xacro:sensor_d455 parent="base_link" use_nominal_extrinsics="$(arg use_nominal_extrinsics)">
+        <origin xyz="0.2 0 0.3" rpy="0 0 0"/>
+    </xacro:sensor_d455>
+    <!-- end sensors -->
 </robot>

Commit message: add more parts to robot model

File: sctebot2_description/urdf/standard/sctebot2.urdf.xacro (robot description, xacro)
@@ -6,5 +6,5 @@
     R2D2 https://github.com/ros/urdf_tutorial/tree/ros2
      -->
-    <!-- Math constants -->
+    <!-- math constants -->
     <xacro:property name="deg_to_rad" value="0.01745329251994329577"/>
     <!-- materials -->
@@ -24,5 +24,5 @@
         <color rgba="0 0.8 0 1"/>
     </material>
-    <!-- Robot base dimensions -->
+    <!-- robot base dimensions -->
     <xacro:property name="base_length" value="0.442" /> <!-- wheel base derived from this -->
     <xacro:property name="base_width" value="0.157" /> <!-- wheel track derived from this -->
@@ -38,5 +38,5 @@
             <origin xyz="0 0 0" rpy="0 0 0"/>
             <geometry>
-                <box size="${base_length} ${base_width} ${base_height}"/>
+                <box size="${base_length} ${base_width} ${base_height * 0.1}"/>
             </geometry>
             <material name="green"/>
@@ -63,4 +63,34 @@
         </collision>
     </link>
+    <!-- base links -->
+    <!-- shock towers -->
+    <xacro:property name="shock_tower_height" value="0.08"/>
+    <link name="front_shocker_tower">
+        <visual>
+            <origin xyz="0 0 0" rpy="0 0 0"/>
+            <geometry>
+                <box size="0.01 0.12 ${shock_tower_height}"/>
+            </geometry>
+        </visual>
+    </link>
+    <joint name="front_shock_tower_base_link" type="fixed">
+        <origin xyz="${wheel_base / 2.0} 0 ${wheel_axis_height}" rpy="0 0 0"/>
+        <parent link="base_link"/>
+        <child link="front_shocker_tower"/>
+    </joint>
+    <link name="rear_shocker_tower">
+        <visual>
+            <origin xyz="0 0 0" rpy="0 0 0"/>
+            <geometry>
+                <box size="0.01 0.12 ${shock_tower_height}"/>
+            </geometry>
+        </visual>
+    </link>
+    <joint name="rear_shock_tower_base_link" type="fixed">
+        <origin xyz="-${wheel_base / 2.0} 0 ${wheel_axis_height}" rpy="0 0 0"/>
+        <parent link="base_link"/>
+        <child link="rear_shocker_tower"/>
+    </joint>
+    <!-- shock towers -->
     <!-- bumpers -->
     <xacro:property name="front_bumper_offset" value="0.075"/>
@@ -110,5 +140,5 @@
         <child link="rear_bumper"/>
     </joint>
-    <!-- end bumpbers -->
+    <!-- bumpbers -->
     <!-- wheels -->
     <link name="left_front_wheel">
@@ -196,10 +226,36 @@
         <child link="right_rear_wheel"/>
     </joint>
-    <!-- end wheels -->
+    <!-- wheels -->
+    <!-- Ackermann
+    https://control.ros.org/humble/doc/ros2_controllers/steering_controllers_library/doc/userdoc.html
+    https://control.ros.org/humble/doc/ros2_controllers/ackermann_steering_controller/doc/userdoc.html
+    -->
+    <!-- computer housing -->
+    <xacro:property name="computer_housing_height" value="0.12"/>
+    <link name="computer_housing">
+        <visual>
+                <origin xyz="0 0 0" rpy="0 0 0"/>
+                <geometry>
+                        <box size="0.30 0.24 ${computer_housing_height}"/>
+                </geometry>
+            <material name="blue"/>
+            <collision>
+                <geometry>
+                        <box size="0.30 0.24 ${computer_housing_height}"/>
+                </geometry>
+            </collision>
+        </visual>
+    </link>
+    <joint name="computer_housing_base_link" type="fixed">
+        <origin xyz="0 0 ${shock_tower_height + 0.075}" rpy="0 0 0"/>
+        <parent link="base_link"/>
+        <child link="computer_housing"/>
+    </joint>
+    <!-- computer housing -->
     <!-- sensors -->
     <!-- x 0.323m span, 0.162m center from axis z -->
     <link name="ydlidar_sensor">
         <visual>
-            <origin xyz="0 0 0.3" rpy="0 0 0"/>
+            <origin xyz="0 0 0" rpy="0 0 0"/>
             <geometry>
                 <!--cylinder length="0.041" radius="0.035"/-->
@@ -209,13 +265,13 @@
     </link>
     <joint name="ydlidar_sensor_joint" type="fixed">
-        <origin xyz="0 0 0" rpy="0 0 0"/>
-        <parent link="base_link"/>
+        <origin xyz="0 0 ${computer_housing_height / 2.0}" rpy="0 0 0"/>
+        <parent link="computer_housing"/>
         <child link="ydlidar_sensor"/>
     </joint>
     <xacro:include filename="$(find realsense2_description)/urdf/_d455.urdf.xacro"/>
     <xacro:arg name="use_nominal_extrinsics" default="false"/>
-    <xacro:sensor_d455 parent="base_link" use_nominal_extrinsics="$(arg use_nominal_extrinsics)">
-        <origin xyz="0.2 0 0.3" rpy="0 0 0"/>
+    <xacro:sensor_d455 parent="computer_housing" use_nominal_extrinsics="$(arg use_nominal_extrinsics)">
+        <origin xyz="0.13 0 ${computer_housing_height / 2.0}" rpy="0 0 0"/>
     </xacro:sensor_d455>
-    <!-- end sensors -->
+    <!-- sensors -->
 </robot>
