Commit message: got carlikebot xacro visual and geometry  wired into sctebot2 xacro. no controller components yet.

File: sctebot2_description/ros2_control/carlikebot.ros2_control.xacro (robot description, xacro)
@@ -4,5 +4,6 @@
     <ros2_control name="${name}" type="system">
       <hardware>
-        <plugin>ros2_control_demo_example_11/CarlikeBotSystemHardware</plugin>
+        <!--plugin>ros2_control_demo_example_11/CarlikeBotSystemHardware</plugin-->
+        <plugin>carlikebot_ros2_demo_controller/CarlikeBotSystemHardware</plugin>
         <param name="example_param_hw_start_duration_sec">0</param>
         <param name="example_param_hw_stop_duration_sec">3.0</param>

File: sctebot2_description/urdf/standard/sctebot2.urdf.xacro (robot description, xacro)
@@ -8,4 +8,5 @@
     <!-- math constants -->
     <xacro:property name="deg_to_rad" value="0.01745329251994329577"/>
+    <xacro:property name="PI" value="3.1415926535897931"/>
     <!-- materials -->
     <material name="black_front">
@@ -231,4 +232,18 @@
     https://control.ros.org/humble/doc/ros2_controllers/ackermann_steering_controller/doc/userdoc.html
     -->
+    <!-- TBD -->
+    <!-- carlikebot ros2_controller
+    https://github.com/ros-controls/ros2_control_demos/tree/master/example_11
+    https://github.com/ros-controls/ros2_control_demos/blob/master/ros2_control_demo_description/carlikebot/urdf/carlikebot_description.urdf.xacro
+    -->
+    <xacro:include filename="$(find sctebot2_description)/urdf/standard/sctebot2_carlike.urdf.xacro"/>
+    <xacro:carlikebot_virtual_wheels
+        prefix=""
+        wheel_base="${wheel_base}"
+        wheel_radius="${wheel_radius}"
+        wheel_height="${wheel_height}"
+        virtual_rear_wheel_parent_link="base_link"
+        virtual_front_wheel_parent_link="base_link"
+    />
     <!-- computer housing -->
     <xacro:property name="computer_housing_height" value="0.12"/>

File: sctebot2_description/urdf/standard/sctebot2_carlike.urdf.xacro (robot description, xacro)
@@ -1,7 +1,15 @@
 <?xml version="1.0" ?>
 <robot xmlns:xacro="http://www.ros.org/wiki/xacro">
-    <xacro:macro name="carlikebot_virtual_wheels" params="name prefix wheelbase base_height virtual_rear_wheel_parent_link virtual_front_wheel_parent_link">
+    <xacro:macro name="carlikebot_virtual_wheels" params="
+        prefix
+        wheel_base
+        wheel_radius
+        wheel_height
+        virtual_rear_wheel_parent_link
+        virtual_front_wheel_parent_link
+    ">
         <material name="invisible">
-            <color rgba="1.0 0.0 0.0 0.0"/>
+            <!--color rgba="0.0 0.0 0.0 0.0"/-->
+            <color rgba="0.0 0.0 0.0 1.0"/>
         </material>
         <!--virtual rear wheel -->
@@ -10,5 +18,5 @@
                 <origin xyz="0 0 0" rpy="0 0 0"/>
                 <geometry>
-                    <cylinder length="0.10" radius="0.10"/>
+                    <cylinder length="${wheel_height}" radius="${wheel_radius}"/>
                 </geometry>
                 <material name="invisible"/>
@@ -18,6 +26,6 @@
             <parent link="${virtual_rear_wheel_parent_link}"/>
             <child link="${prefix}virtual_rear_wheel"/>
-            <origin xyz="-${wheelbase/2} 0 -${base_height/2}" rpy="0 0 ${PI/2}"/>
-            <axis xyz="1 0 0"/>
+            <origin xyz="-${wheel_base/2} 0 0" rpy="${90 * deg_to_rad} 0 0"/>
+            <axis xyz="0 0 1"/>
             <limit effort="100.0" velocity="100.0"/>
             <dynamics damping="0.2"/>
@@ -28,5 +36,5 @@
                 <origin xyz="0 0 0" rpy="0 0 0"/>
                 <geometry>
-                    <cylinder length="0.1" radius="0.1"/>
+                    <cylinder length="${wheel_height}" radius="${wheel_radius}"/>
                 </geometry>
                 <material name="invisible"/>
@@ -36,5 +44,5 @@
             <parent link="${virtual_front_wheel_parent_link}"/>
             <child link="${prefix}virtual_front_wheel"/>
-            <origin xyz="${wheelbase/2} 0 -${base_height/2}" rpy="0 0 ${PI/2}"/>
+            <origin xyz="${wheel_base/2} 0 0" rpy="${90 * deg_to_rad} 0 0"/>
             <axis xyz="0 0 1"/>
             <limit lower="-0.4" upper="0.4" effort="100.0" velocity="10.0"/>
@@ -45,5 +53,5 @@
             <parent link="${prefix}chassis_link" />
             <child link="${prefix}front_left_wheel" />
-            <origin xyz="${wheelbase/2} -${base_width/2} -${base_height/2}" rpy="0 0 ${PI/2}"/>
+            <origin xyz="${wheelbase/2} -${base_width/2} 0" rpy="0 0 ${PI/2}"/>
             <axis xyz="0 0 1"/>
             <limit lower="-0.4" upper="0.4" effort="100.0" velocity="10.0"/>
